Commit message: Add a test node and fix launch files

File: ar3_description/ros2_control/ar3_system_position_only.ros2_control.xacro (robot description, xacro)
@@ -1,12 +1,12 @@
 <?xml version="1.0"?>
 <robot xmlns:xacro="http://www.ros.org/wiki/xacro">
-  <xacro:macro name="ar3_system_position_only" params="name prefix serial_device serial_baudrate firmware_version sim_gazebo:=^|false use_fake_hardware:=^|true fake_sensor_commands:=^|false">
+  <xacro:macro name="ar3_system_position_only" params="name prefix serial_device serial_baudrate firmware_version use_sim:=^|false use_fake_hardware:=^|true fake_sensor_commands:=^|false">
     <ros2_control name="${name}" type="system">
-      <xacro:if value="$(arg sim_gazebo)">
+      <xacro:if value="$(arg use_sim)">
         <hardware>
           <plugin>gazebo_ros2_control/GazeboSystem</plugin>
         </hardware>
       </xacro:if>
-      <xacro:unless value="$(arg sim_gazebo)">
+      <xacro:unless value="$(arg use_sim)">
         <hardware>
           <xacro:if value="${use_fake_hardware}">
